File: REVERB Interface/REVERB Interface.kicad_pcb (KiCad board)
At the start: 2 copper layers, 90.2 x 95.9 mm, 39 parts, among them J1 RPiZeroW, J2 Iridium, J3 APRS, J4 Antenna, J6 USB_B_Micro, J7 USB, M1 MountingHole_Pad, M2 MountingHole_Pad, M3 MountingHole_Pad, M4 MountingHole_Pad, U1 LSM9DS1BOB, U2 MAX3232, U3 CY7C65213-28PVXI

Commit message: finishing up for real now
Parts:
- added J8: USBPOGO, Connector_PinSocket_2.54mm:PinSocket_1x02_P2.54mm_Vertical, F.Cu at (191.0, 98.0)
- added M5: PiMount, MountingHole:MountingHole_2.7mm_M2.5, F.Cu at (167.4, 79.2)
- added M6: PiMount, MountingHole:MountingHole_2.7mm_M2.5, F.Cu at (167.6, 136.6)
- added M7: PiMount, MountingHole:MountingHole_2.7mm_M2.5, F.Cu at (190.7, 78.6)
- added M8: PiMount, MountingHole:MountingHole_2.7mm_M2.5, F.Cu at (190.7, 136.6)
- added TP1: GND, TestPoint:TestPoint_Pad_D2.0mm, F.Cu at (182.9, 70.1)
- added TP2: 3V3, TestPoint:TestPoint_Pad_D2.0mm, F.Cu at (153.9, 70.6)
- added TP3: 5V, TestPoint:TestPoint_Pad_D2.0mm, F.Cu at (149.9, 70.6)
- added TP4: BAT, TestPoint:TestPoint_Pad_D2.0mm, F.Cu at (179.3, 70.1)
- added TP5: 12V, TestPoint:TestPoint_Pad_D2.0mm, F.Cu at (145.8, 70.6)
- moved C8 17.8 mm to (149.9, 136.5), turned to 270 degrees
Routing:
- net /D+: track 30.2 -> 79.8 mm
- net /D-: track 31.1 -> 73.7 mm
- net +5V: track 95.2 -> 108.4 mm
- net +12V: track 2.54 -> 13.9 mm
- net +3V3: track 2.54 -> 13.7 mm, vias 0 -> 1
- net VBUS: track 2.54 -> 13.3 mm
- net Net-(C8-Pad1): track 7.58 -> 11.4 mm, vias 0 -> 2
- net GND: track 32.3 -> 34.4 mm, vias 16 -> 18
Other:
- board text added: "12V"
- board text added: "3V3"
- board text added: "5V"
- board text added: "BAT"
- board text added: "D+"
- board text added: "D-"
- board text added: "Set JP1 same as JP2 and JP3 same as JP4 JP3 and JP4 should be opposite JP1 and JP2"
