File: REVERB Interface SPI/REVERB Interface.sch (KiCad schematic (older format))
At the start: 49 parts, among them J1 RPiZeroW, J2 Iridium, J3 APRS, J4 Antenna, J6 USB_B_Micro, J7 USB, J8 USBPOGO, M1 MountingHole_Pad, M2 MountingHole_Pad, M3 MountingHole_Pad, M4 MountingHole_Pad, M5 PiMount, M6 PiMount, M7 PiMount, M8 PiMount, U1 LSM9DS1BOB, U2 MAX3232, U3 CY7C65213-28PVXI

Commit message: fix a via
Parts:
- removed J6: USB_B_Micro, REVERB Interface:AdafruitMicroB, symbol Connector:USB_B_Micro
- removed J7: USB, Connector_PinSocket_2.54mm:PinSocket_1x02_P2.54mm_Vertical, symbol Connector:Conn_01x02_Male
- removed J8: USBPOGO, Connector_PinSocket_2.54mm:PinSocket_1x02_P2.54mm_Vertical, symbol Connector:Conn_01x02_Male
- removed U3: CY7C65213-28PVXI, Package_SO:SSOP-28_5.3x10.2mm_P0.65mm, symbol Interface_USB:CY7C65213-28PVXI
- added U?: SC16IS752IPW, Package_SO:TSSOP-28_4.4x9.7mm_P0.65mm, symbol Interface_UART:SC16IS752IPW
- added U?: SC16IS750xPW, Package_SO:TSSOP-24_4.4x7.8mm_P0.65mm, symbol Interface_UART:SC16IS750xPW
- JP3: value USBUARTRX -> SPIUARTRX
- JP4: value USBUARTTX -> SPIUARTTX
Connections:
- net labels added: SPIUARTRX, SPIUARTTX
- net labels removed: D+, D-, USBUARTRX, USBUARTTX
- wire segments 97 -> 92
- no-connect marks 96 -> 95
Other:
- note added: "SPI TO UART"
- note removed: "Micro B for programming"
- note removed: "USB TO UART"
- moved on the sheet: C8, D1, D2, R1, R2
Changed lines of the file:
@@
 $EndComp
-$Comp
-L Connector:Conn_01x02_Male J7
-U 1 1 615C5D8E
-P 6950 1800
-F 0 "J7" H 7058 1981 50  0000 C CNN
-F 1 "USB" H 7058 1890 50  0000 C CNN
-F 2 "Connector_PinSocket_2.54mm:PinSocket_1x02_P2.54mm_Vertical" H 6950 1800 50  0001 C CNN
-F 3 "~" H 6950 1800 50  0001 C CNN
-	1    6950 1800
-	1    0    0    -1
-$EndComp
-Text Label 7150 1800 0    50   ~ 0
-D+
-Text Label 7150 1900 0    50   ~ 0
-D-
 $Comp
 L Interface_UART:MAX3232 U2
@@
 	1    0    0    -1
 $EndComp
-Text Label 3550 4500 0    50   ~ 0
-D+
-Text Label 3550 4600 0    50   ~ 0
-D-
-Text Label 2400 4000 0    50   ~ 0
+Text Label 2600 4200 0    50   ~ 0
 SW7
 $Comp
 L power:GND #PWR0123
 U 1 1 615E7235
-P 2950 5900
-F 0 "#PWR0123" H 2950 5650 50  0001 C CNN
-F 1 "GND" H 2955 5727 50  0000 C CNN
-F 2 "" H 2950 5900 50  0001 C CNN
-F 3 "" H 2950 5900 50  0001 C CNN
-	1    2950 5900
-	1    0    0    -1
-$EndComp
-Text Label 1550 4800 2    50   ~ 0
-USBUARTTX
-Text Label 1550 4700 2    50   ~ 0
-USBUARTRX
+P -3900 5500
+F 0 "#PWR0123" H -3900 5250 50  0001 C CNN
+F 1 "GND" H -3895 5327 50  0000 C CNN
+F 2 "" H -3900 5500 50  0001 C CNN
+F 3 "" H -3900 5500 50  0001 C CNN
+	1    -3900 5500
+	1    0    0    -1
+$EndComp
+Text Label 1400 4750 2    50   ~ 0
+SPIUARTTX
+Text Label 1400 4650 2    50   ~ 0
+SPIUARTRX
 Text Label 7400 4250 0    50   ~ 0
 SW6
@@
 Text Label 5100 1750 2    50   ~ 0
 SPICE0
-$Comp
-L Interface_USB:CY7C65213-28PVXI U3
-U 1 1 61646441
-P 2950 5100
-F 0 "U3" H 3000 6081 50  0000 C CNN
-F 1 "CY7C65213-28PVXI" H 3000 5990 50  0000 C CNN
-F 2 "Package_SO:SSOP-28_5.3x10.2mm_P0.65mm" H 2950 4200 50  0001 C CNN
-F 3 "http://www.cypress.com/file/139881/download" H 450 5600 50  0001 C CNN
-	1    2950 5100
-	1    0    0    -1
-$EndComp
-Wire Wire Line
-	3050 4300 2950 4300
-Wire Wire Line
-	2850 5900 2950 5900
-Connection ~ 2950 5900
-Wire Wire Line
-	2950 5900 3050 5900
+Wire Wire Line
+	-800 4350 -900 4350
 $Comp
 L Device:C C7
@@
 	1    0    0    -1
 $EndComp
-Text Label 1950 5950 1    50   ~ 0
+Text Label -1900 6000 1    50   ~ 0
 SW7
 $Comp
@@
 L Device:C C8
 U 1 1 6166454E
-P 2150 5700
-F 0 "C8" H 2265 5746 50  0000 L CNN
-F 1 "1uF" H 2265 5655 50  0000 L CNN
-F 2 "Capacitor_SMD:C_0805_2012Metric_Pad1.18x1.45mm_HandSolder" H 2188 5550 50  0001 C CNN
-F 3 "~" H 2150 5700 50  0001 C CNN
-	1    2150 5700
-	1    0    0    -1
-$EndComp
-Wire Wire Line
-	2850 5900 2150 5900
-Wire Wire Line
-	2150 5900 2150 5850
-Connection ~ 2850 5900
-Wire Wire Line
-	2450 5500 2150 5500
-Wire Wire Line
-	2150 5500 2150 5550
-$Comp
-L Connector:USB_B_Micro J6
-U 1 1 6166AFCB
-P 1150 5400
-F 0 "J6" H 1207 5867 50  0000 C CNN
-F 1 "USB_B_Micro" H 1207 5776 50  0000 C CNN
-F 2 "REVERB Interface:AdafruitMicroB" H 1300 5350 50  0001 C CNN
-F 3 "~" H 1300 5350 50  0001 C CNN
-	1    1150 5400
-	1    0    0    -1
-$EndComp
-Text Label 1450 5200 0    50   ~ 0
-SW7
-Text Label 1450 5400 0    50   ~ 0
-D+
-Text Label 1450 5500 0    50   ~ 0
-D-
-NoConn ~ 1450 5600
-Wire Wire Line
-	1050 5800 1150 5800
-Wire Wire Line
-	1450 5800 1450 5900
-Connection ~ 1150 5800
-Wire Wire Line
-	1150 5800 1450 5800
-$Comp
-L power:GND #PWR0128
-U 1 1 61672E01
-P 1450 5900
-F 0 "#PWR0128" H 1450 5650 50  0001 C CNN
-F 1 "GND" H 1455 5727 50  0000 C CNN
-F 2 "" H 1450 5900 50  0001 C CNN
-F 3 "" H 1450 5900 50  0001 C CNN
-	1    1450 5900
-	1    0    0    -1
-$EndComp
-Wire Wire Line
-	2450 4700 1650 4700
-Wire Wire Line
-	2450 4800 2050 4800
+P -1700 5750
+F 0 "C8" H -1585 5796 50  0000 L CNN
+F 1 "1uF" H -1585 5705 50  0000 L CNN
+F 2 "Capacitor_SMD:C_0805_2012Metric_Pad1.18x1.45mm_HandSolder" H -1662 5600 50  0001 C CNN
+F 3 "~" H -1700 5750 50  0001 C CNN
+	1    -1700 5750
+	1    0    0    -1
+$EndComp
+Wire Wire Line
+	-1700 5950 -1700 5900
+Wire Wire Line
+	-1400 5550 -1700 5550
+Wire Wire Line
+	-1700 5550 -1700 5600
+Wire Wire Line
+	-1400 4750 -2200 4750
+Wire Wire Line
+	-1400 4850 -1800 4850
 $Comp
 L Device:LED D1
 U 1 1 61680797
-P 2050 4450
-F 0 "D1" V 2089 4332 50  0000 R CNN
-F 1 "RED" V 1998 4332 50  0000 R CNN
-F 2 "LED_SMD:LED_0805_2012Metric_Pad1.15x1.40mm_HandSolder" H 2050 4450 50  0001 C CNN
-F 3 "~" H 2050 4450 50  0001 C CNN
-	1    2050 4450
+P -1800 4500
+F 0 "D1" V -1761 4382 50  0000 R CNN
+F 1 "RED" V -1852 4382 50  0000 R CNN
+F 2 "LED_SMD:LED_0805_2012Metric_Pad1.15x1.40mm_HandSolder" H -1800 4500 50  0001 C CNN
+F 3 "~" H -1800 4500 50  0001 C CNN
+	1    -1800 4500
 	0    -1   -1   0
 $EndComp
@@
 L Device:LED D2
 U 1 1 61681979
-P 1650 4450
-F 0 "D2" V 1689 4332 50  0000 R CNN
-F 1 "GREEN" V 1598 4332 50  0000 R CNN
-F 2 "LED_SMD:LED_0805_2012Metric_Pad1.15x1.40mm_HandSolder" H 1650 4450 50  0001 C CNN
-F 3 "~" H 1650 4450 50  0001 C CNN
-	1    1650 4450
+P -2200 4500
+F 0 "D2" V -2161 4382 50  0000 R CNN
+F 1 "GREEN" V -2252 4382 50  0000 R CNN
+F 2 "LED_SMD:LED_0805_2012Metric_Pad1.15x1.40mm_HandSolder" H -2200 4500 50  0001 C CNN
+F 3 "~" H -2200 4500 50  0001 C CNN
+	1    -2200 4500
 	0    -1   -1   0
 $EndComp
@@
 L Device:R R1
 U 1 1 61683EE4
-P 2050 4150
-F 0 "R1" V 1950 4100 50  0000 L CNN
-F 1 "1K" V 2050 4100 50  0000 L CNN
-F 2 "Resistor_SMD:R_0805_2012Metric_Pad1.20x1.40mm_HandSolder" V 1980 4150 50  0001 C CNN
-F 3 "~" H 2050 4150 50  0001 C CNN
-	1    2050 4150
+P -1800 4200
+F 0 "R1" V -1900 4150 50  0000 L CNN
+F 1 "1K" V -1800 4150 50  0000 L CNN
+F 2 "Resistor_SMD:R_0805_2012Metric_Pad1.20x1.40mm_HandSolder" V -1870 4200 50  0001 C CNN
+F 3 "~" H -1800 4200 50  0001 C CNN
+	1    -1800 4200
 	1    0    0    -1
 $EndComp
@@
 L Device:R R2
 U 1 1 6168462F
-P 1650 4150
-F 0 "R2" V 1550 4100 50  0000 L CNN
-F 1 "1K" V 1650 4100 50  0000 L CNN
-F 2 "Resistor_SMD:R_0805_2012Metric_Pad1.20x1.40mm_HandSolder" V 1580 4150 50  0001 C CNN
-F 3 "~" H 1650 4150 50  0001 C CNN
-	1    1650 4150
-	1    0    0    -1
-$EndComp
-Wire Wire Line
-	1650 4000 2050 4000
-Connection ~ 2050 4000
-Wire Wire Line
-	2050 4600 2050 4800
-Connection ~ 2050 4800
-Wire Wire Line
-	2050 4800 1550 4800
-Wire Wire Line
-	1650 4600 1650 4700
-Connection ~ 1650 4700
-Wire Wire Line
-	1650 4700 1550 4700
-Wire Wire Line
-	2950 4300 2950 4000
-Wire Wire Line
-	2050 4000 2950 4000
-Connection ~ 2950 4300
+P -2200 4200
+F 0 "R2" V -2300 4150 50  0000 L CNN
+F 1 "1K" V -2200 4150 50  0000 L CNN
+F 2 "Resistor_SMD:R_0805_2012Metric_Pad1.20x1.40mm_HandSolder" V -2270 4200 50  0001 C CNN
+F 3 "~" H -2200 4200 50  0001 C CNN
+	1    -2200 4200
+	1    0    0    -1
+$EndComp
+Wire Wire Line
+	-2200 4050 -1800 4050
+Connection ~ -1800 4050
+Wire Wire Line
+	-1800 4650 -1800 4850
+Connection ~ -1800 4850
+Wire Wire Line
+	-1800 4850 -2300 4850
+Wire Wire Line
+	-2200 4650 -2200 4750
+Connection ~ -2200 4750
+Wire Wire Line
+	-2200 4750 -2300 4750
+Wire Wire Line
+	-900 4350 -900 4050
+Wire Wire Line
+	-1800 4050 -900 4050
 $Comp
 L Device:LED D3
@@
 Wire Wire Line
 	4200 5850 4750 5850
-Text Notes 900  4900 0    50   ~ 0
-Micro B for programming
 Text Notes 850  4000 0    50   ~ 0
-USB TO UART
+SPI TO UART
 Wire Notes Line
 	850  3900 3700 3900
@@
 APRSRX
 Text Label 10650 2950 3    50   ~ 0
-USBUARTTX
+SPIUARTTX
 Text Label 8550 2950 3    50   ~ 0
-USBUARTRX
+SPIUARTRX
 $Comp
 L Jumper:SolderJumper_3_Open JP3
@@
 P 8550 2800
 F 0 "JP3" H 8550 3005 50  0000 C CNN
-F 1 "USBUARTRX" H 8550 2914 50  0000 C CNN
+F 1 "SPIUARTRX" H 8550 2914 50  0000 C CNN
 F 2 "Jumper:SolderJumper-3_P1.3mm_Open_Pad1.0x1.5mm_NumberLabels" H 8550 2800 50  0001 C CNN
 F 3 "~" H 8550 2800 50  0001 C CNN
@@
 P 10650 2800
 F 0 "JP4" H 10650 3005 50  0000 C CNN
-F 1 "USBUARTTX" H 10650 2914 50  0000 C CNN
+F 1 "SPIUARTTX" H 10650 2914 50  0000 C CNN
 F 2 "Jumper:SolderJumper-3_P1.3mm_Open_Pad1.0x1.5mm_NumberLabels" H 10650 2800 50  0001 C CNN
 F 3 "~" H 10650 2800 50  0001 C CNN
@@
 	3750 3900 6950 3900
 $Comp
-L Connector:Conn_01x02_Male J8
-U 1 1 61634D7E
-P 7450 1800
-F 0 "J8" H 7558 1981 50  0000 C CNN
-F 1 "USBPOGO" H 7558 1890 50  0000 C CNN
-F 2 "Connector_PinSocket_2.54mm:PinSocket_1x02_P2.54mm_Vertical" H 7450 1800 50  0001 C CNN
-F 3 "~" H 7450 1800 50  0001 C CNN
-	1    7450 1800
-	1    0    0    -1
-$EndComp
-Text Label 7650 1800 0    50   ~ 0
-D+
-Text Label 7650 1900 0    50   ~ 0
-D-
-$Comp
 L Mechanical:MountingHole M5
 U 1 1 61640E3F
@@
 	0    -1   -1   0
 $EndComp
+$Comp
+L Interface_UART:SC16IS752IPW U?
+U 1 1 6164DB56
+P -3900 4500
+F 0 "U?" H -3900 5681 50  0000 C CNN
+F 1 "SC16IS752IPW" H -3900 5590 50  0000 C CNN
+F 2 "Package_SO:TSSOP-28_4.4x9.7mm_P0.65mm" H -3900 2950 50  0001 C CNN
+F 3 "https://www.nxp.com/docs/en/data-sheet/SC16IS752_SC16IS762.pdf" H -3900 3100 50  0001 C CNN
+	1    -3900 4500
+	1    0    0    -1
+$EndComp
+Wire Wire Line
+	2150 5900 3050 5900
+$Comp
+L Interface_UART:SC16IS750xPW U?
+U 1 1 61657D27
+P -2150 2950
+F 0 "U?" H -2150 4031 50  0000 C CNN
+F 1 "SC16IS750xPW" H -2150 3940 50  0000 C CNN
+F 2 "Package_SO:TSSOP-24_4.4x7.8mm_P0.65mm" H -2150 1650 50  0001 C CNN
+F 3 "https://www.nxp.com/docs/en/data-sheet/SC16IS740_750_760.pdf" H -50 3300 50  0001 C CNN
+	1    -2150 2950
+	1    0    0    -1
+$EndComp
 $EndSCHEMATC

Commit message: spi edits
Parts:
- removed U?: SC16IS750xPW, Package_SO:TSSOP-24_4.4x7.8mm_P0.65mm, symbol Interface_UART:SC16IS750xPW
- added C9: 33pF, Capacitor_SMD:C_0805_2012Metric_Pad1.18x1.45mm_HandSolder, symbol Device:C
- added R7, R8: 1K, Resistor_SMD:R_0805_2012Metric_Pad1.20x1.40mm_HandSolder, symbol Device:R
- added Y1: 1.8432MHz, Crystal:Crystal_HC49-U_Vertical, symbol Device:Crystal
- C6: value 4.7uF -> 10uF
- C8: value 1uF -> 22pF
- gave numbers to parts that had none: 1
Connections:
- net labels added: CTS, RTS
- wire segments 92 -> 100
Other:
- note added: "Option 1: Hardware APRS, two converters to Iridium: \nJP1 and JP2 bridge pins 2 and 3, JP3 and JP4 bridge pins 1 and 2\nOption 2: SPI UART APRS, MAX3232 Iridium:\nJP1 and JP2 bridge pins 1 and 2, JP3 and JP4 bridge pins 2 and 3\nDO NOT BRIDGE THE SAME TWO PINS FOR BOTH PAIRS OF JUMPERS"
- note removed: "Option 1: Hardware APRS, two converters to Iridium: \nJP1 and JP2 bridge pins 2 and 3, JP3 and JP4 bridge pins 1 and 2\nOption 2: USB UART APRS, MAX3232 Iridium:\nJP1 and JP2 bridge pins 1 and 2, JP3 and JP4 bridge pins 2 and 3\nDO NOT BRIDGE THE SAME TWO PINS FOR BOTH PAIRS OF JUMPERS"
- moved on the sheet: C1, C2, C3, C4, C5, C6, C7, D1, D2, D3, D4, D5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
